Commit message: Working run commads to see working

File: install/rarm/share/rarm/urdf/GP7.urdf.xacro (robot description, xacro)
@@ -3,4 +3,27 @@
     <xacro:property name="joint_damping" value="5.0"/>
   <xacro:property name="joint_friction" value="0.3"/>
+<xacro:macro name="friction_details">
+<!-- Added New -->
+        <surface>
+    <friction>
+      <ode>
+        <mu>5.0</mu>    <!-- primary friction -->
+        <mu2>5.0</mu2>  <!-- secondary friction -->
+      </ode>
+    </friction>
+    <contact>
+      <ode>
+        <kp>100000</kp>   <!-- contact stiffness -->
+        <kd>1.0</kd>      <!-- contact damping -->
+        <max_vel>0.1</max_vel>      <!-- optional: max contact velocity -->
+        <min_depth>0.001</min_depth> <!-- optional: penetration depth limit -->
+      </ode>
+    </contact>
+    <bounce>
+      <restitution_coefficient>0.0</restitution_coefficient> <!-- no bouncing -->
+    </bounce>
+  </surface>
+     <!-- Added New -->
+</xacro:macro>
    <link name="world"/>
   <joint
@@ -166,11 +189,11 @@
       link="L2" />
     <axis
-      xyz="0 0 -1" />
-    <limit
-      lower="-2.53"
-      upper="1.135"
-      effort="30"
+      xyz="0 0 1" />
+    <limit
+      lower="-1.135"
+      upper="2.53"
+      effort="100"
       velocity="5.497" />
-        <dynamics damping="${joint_damping}" friction="${joint_friction}"/>
+      <dynamics damping="${joint_damping}" friction="${joint_friction}"/>
   </joint>
   <link
@@ -227,6 +250,6 @@
       xyz="0 0 1" />
     <limit
-      lower="-1.222"
-      upper="3.316"
+      upper="1.222"
+      lower="-3.316"
       effort="30"
       velocity="7.155" />
@@ -404,5 +427,5 @@
       xyz="0 0 1" />
     <limit
-      lower="0"
+      lower="-6.2832"
       upper="6.2832"
       effort="30"
@@ -448,4 +471,5 @@
           filename="package://rarm/meshes/L7.STL" />
       </geometry>
+      <xacro:friction_details/>
     </collision>
   </link>
@@ -507,4 +531,5 @@
           filename="package://rarm/meshes/L8.STL" />
       </geometry>
+         <xacro:friction_details/>
     </collision>
   </link>

File: install/rarm/share/rarm/urdf/GP7_ros2_control.urdf.xacro (robot description, xacro)
@@ -17,6 +17,6 @@
             <joint name="J2">
                 <command_interface name="position">
-                    <param name="min">-2.53</param>
-                    <param name="max">1.135</param>
+                    <param name="min">-1.135</param>
+                    <param name="max">2.53</param>
                 </command_interface>
                 <state_interface name="position"/>
@@ -24,6 +24,6 @@
             <joint name="J3">
                 <command_interface name="position">
-                    <param name="min">-1.222</param>
-                    <param name="max">3.316</param>
+                    <param name="min">-3.316</param>
+                    <param name="max">1.222</param>
                 </command_interface>
                 <state_interface name="position"/>
@@ -45,5 +45,5 @@
             <joint name="J6">
                 <command_interface name="position">
-                    <param name="min">0</param>
+                    <param name="min">-6.2832</param>
                     <param name="max">6.2832</param>
                 </command_interface>

Commit message: not working dont merge

File: install/rarm/share/rarm/urdf/GP7.urdf.xacro (robot description, xacro)
@@ -440,5 +440,5 @@
         rpy="0 0 0" />
       <mass
-        value="0.040444" />
+        value="0.04" />
       <inertia
         ixx="5.0254E-05"
@@ -451,9 +451,10 @@
     <visual>
       <origin
-        xyz="0 0 0"
-        rpy="0 0 0" />
-      <geometry>
-        <mesh
-          filename="package://rarm/meshes/L7.STL" />
+        xyz="-0.01 0.08 0"
+        rpy="0 0 0" />
+      <geometry>
+        <!-- <mesh
+          filename="package://rarm/meshes/L7.STL" /> -->
+          <box size="0.06 0.140 0.06" />
       </geometry>
       <material
@@ -465,9 +466,10 @@
     <collision>
       <origin
-        xyz="0 0 0"
-        rpy="0 0 0" />
-      <geometry>
-        <mesh
-          filename="package://rarm/meshes/L7.STL" />
+        xyz="-0.01 0.08 0"
+        rpy="0 0 0" />
+      <geometry>
+        <!-- <mesh
+          filename="package://rarm/meshes/L7.STL" /> -->
+          <box size="0.06 0.140 0.06" />
       </geometry>
       <xacro:friction_details/>
@@ -476,5 +478,5 @@
   <joint
     name="J7"
-    type="revolute">
+    type="prismatic">
     <origin
       xyz="0 0.044379 0.11015"
@@ -485,7 +487,7 @@
       link="L7" />
     <axis
-      xyz="0 0 -1" />
-    <limit
-      lower="-1.57"
+      xyz="1 0 0" />
+    <limit
+      lower="-0.05"
       upper="0"
       effort="30"
@@ -500,5 +502,5 @@
         rpy="0 0 0" />
       <mass
-        value="0.040444" />
+        value="0.04" />
       <inertia
         ixx="5.0254E-05"
@@ -511,9 +513,10 @@
     <visual>
       <origin
-        xyz="0 0 0"
-        rpy="0 0 0" />
-      <geometry>
-        <mesh
-          filename="package://rarm/meshes/L8.STL" />
+        xyz="0 0.08 0"
+        rpy="0 0 0" />
+      <geometry>
+        <!-- <mesh
+          filename="package://rarm/meshes/L8.STL" /> -->
+          <box size="0.06 0.140 0.06" />
       </geometry>
       <material
@@ -525,9 +528,10 @@
     <collision>
       <origin
-        xyz="0 0 0"
-        rpy="0 0 0" />
-      <geometry>
-        <mesh
-          filename="package://rarm/meshes/L8.STL" />
+        xyz="0 0.08 0"
+        rpy="0 0 0" />
+      <geometry>
+        <!-- <mesh
+          filename="package://rarm/meshes/L8.STL" /> -->
+          <box size="0.06 0.140 0.06" />
       </geometry>
          <xacro:friction_details/>
@@ -536,5 +540,5 @@
   <joint
     name="J8"
-    type="revolute">
+    type="prismatic">
     <origin
       xyz="0 -0.044379 0.11015"
@@ -545,11 +549,11 @@
       link="L8" />
     <axis
-      xyz="0 0 1" />
-    <limit
-      lower="-1.57"
-      upper="0"
+      xyz="1 0 0" />
+    <limit
+      lower="0"
+      upper="0.05"
       effort="30"
       velocity="10" />
-      <mimic joint="J7" multiplier="1.0" offset="0"/>
+       <mimic joint="J7" multiplier="-1.0" offset="0"/>
        <dynamics damping="${joint_damping}" friction="${joint_friction}"/>
   </joint>

File: install/rarm/share/rarm/urdf/GP7_ros2_control.urdf.xacro (robot description, xacro)
@@ -52,5 +52,5 @@
             <joint name="J7">
                 <command_interface name="position">
-                    <param name="min">-1.57</param>
+                    <param name="min">-0.05</param>
                     <param name="max">0</param>
                 </command_interface>
@@ -60,5 +60,5 @@
             <joint name="J8">
                 <param name="mimic">J7</param>
-                <param name="multiplier">1.0</param>
+                <param name="multiplier">-1.0</param>
                 <state_interface name="position"/>
                 <state_interface name="velocity"/>

Commit message: Done merge to main

File: install/rarm/share/rarm/urdf/GP7.urdf.xacro (robot description, xacro)
@@ -440,5 +440,5 @@
         rpy="0 0 0" />
       <mass
-        value="0.04" />
+        value="0.040444" />
       <inertia
         ixx="5.0254E-05"
@@ -451,10 +451,9 @@
     <visual>
       <origin
-        xyz="-0.01 0.08 0"
-        rpy="0 0 0" />
-      <geometry>
-        <!-- <mesh
-          filename="package://rarm/meshes/L7.STL" /> -->
-          <box size="0.06 0.140 0.06" />
+        xyz="-0.01 0 0"
+        rpy="0 0 0" />
+      <geometry>
+        <mesh
+          filename="package://rarm/meshes/L7.STL" />
       </geometry>
       <material
@@ -466,10 +465,9 @@
     <collision>
       <origin
-        xyz="-0.01 0.08 0"
-        rpy="0 0 0" />
-      <geometry>
-        <!-- <mesh
-          filename="package://rarm/meshes/L7.STL" /> -->
-          <box size="0.06 0.140 0.06" />
+        xyz="-0.01 0 0"
+        rpy="0 0 0" />
+      <geometry>
+        <mesh
+          filename="package://rarm/meshes/L7.STL" />
       </geometry>
       <xacro:friction_details/>
@@ -502,5 +500,5 @@
         rpy="0 0 0" />
       <mass
-        value="0.04" />
+        value="0.040444" />
       <inertia
         ixx="5.0254E-05"
@@ -513,10 +511,9 @@
     <visual>
       <origin
-        xyz="0 0.08 0"
-        rpy="0 0 0" />
-      <geometry>
-        <!-- <mesh
-          filename="package://rarm/meshes/L8.STL" /> -->
-          <box size="0.06 0.140 0.06" />
+        xyz="0 0 0"
+        rpy="0 0 0" />
+      <geometry>
+        <mesh
+          filename="package://rarm/meshes/L8.STL" />
       </geometry>
       <material
@@ -528,10 +525,9 @@
     <collision>
       <origin
-        xyz="0 0.08 0"
-        rpy="0 0 0" />
-      <geometry>
-        <!-- <mesh
-          filename="package://rarm/meshes/L8.STL" /> -->
-          <box size="0.06 0.140 0.06" />
+        xyz="0 0 0"
+        rpy="0 0 0" />
+      <geometry>
+        <mesh
+          filename="package://rarm/meshes/L8.STL" />
       </geometry>
          <xacro:friction_details/>
